Commit message: more gripper fixes

File: src/igus_rebel_ros2/src/igus_rebel_description/urdf/igus_rebel2.urdf (robot description, URDF)
Before this commit: robot igus_rebel, 16 links, 15 joints
Joints:
- joint gripper_l_joint: type prismatic -> fixed
- joint gripper_r_joint: type prismatic -> fixed

Commit message: reduced meshes

File: src/igus_rebel_ros2/src/igus_rebel_description/urdf/igus_rebel2.urdf (robot description, URDF)
Before this commit: robot igus_rebel, 16 links, 15 joints
Links:
- link base_link: geometry collision cylinder length=0.1 radius=0.09; visual mesh filename=file://$(find igus_rebel_description)/meshes/IgusMeshes/old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
- link link1: geometry collision box size=0.1 0.03 0.1; visual mesh filename=file://$(find igus_rebel_description)/meshes/IgusMeshes/old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
- link link2: geometry collision cylinder length=0.18 radius=0.06; visual mesh filename=file://$(find igus_rebel_description)/meshes/IgusMeshes/old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
- link link3: geometry collision box size=0.1 0.03 0.1; visual mesh filename=file://$(find igus_rebel_description)/meshes/IgusMeshes/old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
- link link4: geometry collision cylinder length=0.1 radius=0.05; visual mesh filename=file://$(find igus_rebel_description)/meshes/IgusMeshes/old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
- link link5: geometry collision box size=0.1 0.03 0.1; visual mesh filename=file://$(find igus_rebel_description)/meshes/IgusMeshes/old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
- link link6: geometry collision cylinder length=0.065 radius=0.04; visual mesh filename=file://$(find igus_rebel_description)/meshes/IgusMeshes/old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
- link motor1: geometry collision cylinder length=0.065 radius=0.05; visual mesh filename=file://$(find igus_rebel_description)/meshes/IgusMeshes/old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
- link motor2: geometry collision cylinder length=0.065 radius=0.05; visual mesh filename=file://$(find igus_rebel_description)/meshes/IgusMeshes/old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
- link motor3: geometry collision cylinder length=0.065 radius=0.05; visual mesh filename=file://$(find igus_rebel_description)/meshes/IgusMeshes/old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
- link motor4: geometry collision cylinder length=0.065 radius=0.05; visual mesh filename=file://$(find igus_rebel_description)/meshes/IgusMeshes/old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
- link motor5: geometry collision cylinder length=0.065 radius=0.04; visual mesh filename=file://$(find igus_rebel_description)/meshes/IgusMeshes/old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

Commit message: gripper impl

File: src/igus_rebel_ros2/src/igus_rebel_description/urdf/igus_rebel2.urdf (robot description, URDF)
Before this commit: robot igus_rebel, 16 links, 15 joints
Links:
- link base_link: geometry collision cylinder length=0.1 radius=0.09; visual mesh filename=file://$(find igus_rebel_description)/meshes/IgusMeshes/bas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
- link gripper_base: geometry collision box size=0.1 0.13 0.08; visual mesh filename=file://$(find igus_rebel_description)/meshes/IgusMeshes/gri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 scale=0.001 0.001 0.001
- link link1: geometry collision box size=0.1 0.03 0.1; visual mesh filename=file://$(find igus_rebel_description)/meshes/IgusMeshes/lin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
- link link2: geometry collision cylinder length=0.18 radius=0.06; visual mesh filename=file://$(find igus_rebel_description)/meshes/IgusMeshes/lin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
- link link3: geometry collision box size=0.1 0.03 0.1; visual mesh filename=file://$(find igus_rebel_description)/meshes/IgusMeshes/lin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
- link link4: geometry collision cylinder length=0.1 radius=0.05; visual mesh filename=file://$(find igus_rebel_description)/meshes/IgusMeshes/lin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
- link link5: geometry collision box size=0.1 0.03 0.1; visual mesh filename=file://$(find igus_rebel_description)/meshes/IgusMeshes/lin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
- link link6: geometry collision cylinder length=0.065 radius=0.04; visual mesh filename=file://$(find igus_rebel_description)/meshes/IgusMeshes/lin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
- link motor1: geometry collision cylinder length=0.065 radius=0.05; visual mesh filename=file://$(find igus_rebel_description)/meshes/IgusMeshes/mot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
- link motor2: geometry collision cylinder length=0.065 radius=0.05; visual mesh filename=file://$(find igus_rebel_description)/meshes/IgusMeshes/mot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
- link motor3: geometry collision cylinder length=0.065 radius=0.05; visual mesh filename=file://$(find igus_rebel_description)/meshes/IgusMeshes/mot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
- link motor4: geometry collision cylinder length=0.065 radius=0.05; visual mesh filename=file://$(find igus_rebel_description)/meshes/IgusMeshes/mot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
- link motor5: geometry collision cylinder length=0.065 radius=0.04; visual mesh filename=file://$(find igus_rebel_description)/meshes/IgusMeshes/mot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

Commit message: camera

File: src/igus_rebel_ros2/src/igus_rebel_description/urdf/igus_rebel2.urdf (robot description, URDF)
Before this commit: robot igus_rebel, 16 links, 15 joints
Links:
- added link camera_link; collision box size=0.09 0.025 0.025; visual mesh filename=file://$(find igus_rebel_description)/meshes/IgusMeshes/cam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 scale=0.001 0.001 0.001
- link gripper_base: geometry collision box size=0.09 0.10 0.08; visual mesh filename=file://$(find igus_rebel_description)/meshes/IgusMeshes/gri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 scale=0.001 0.001 0.001
Joints:
- added joint link6_to_camera: type fixed, parent link6, child camera_link, origin xyz=-0.066 0 0 rpy=0 -1.57 0

Commit message: realsense orientation fix

File: src/igus_rebel_ros2/src/igus_rebel_description/urdf/igus_rebel2.urdf (robot description, URDF)
Before this commit: robot igus_rebel, 17 links, 16 joints
Links:
- link camera_link: geometry visual mesh filename=file://$(find igus_rebel_description)/meshes/IgusMeshes/cam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 scale=0.001 0.001 0.001
Joints:
- removed joint link6_to_camera
- added joint link5_to_camera: type fixed, parent link5, child camera_link, origin xyz=0 0 0.05 rpy=0 -1.57 -3.14

Commit message: puck detection, urdf fix

File: src/igus_rebel_ros2/src/igus_rebel_description/urdf/igus_rebel2.urdf (robot description, URDF)
Before this commit: robot igus_rebel, 17 links, 16 joints
Joints:
- joint link5_to_camera: origin xyz=0 0 0.05 rpy=0 -1.57 -3.14 -> xyz=0.068 0 0.093 rpy=0 -1.57 -3.14
